Commit message: add v_slam

File: urdf/bottle_car.urdf.xacro (robot description, xacro)
@@ -1,6 +1,5 @@
 <?xml version="1.0"?>
 <robot name="bottle_car" xmlns:xacro="http://www.ros.org/wiki/xacro">
-    <!-- ======================= PROPERTIES ======================= -->
-    <!-- These values are tuned to look like the image. You can change them here! -->
+    <!-- ================= Properties ================= -->
     <xacro:property name="bottle_length" value="0.22"/>
     <xacro:property name="bottle_radius" value="0.035"/>
@@ -11,36 +10,35 @@
     <xacro:property name="caster_radius" value="0.015"/>
     <xacro:property name="caster_mass" value="0.05"/>
-    <!-- ======================== LINKS (The Physical Parts) ======================== -->
-    <!-- The main body of the car (the bottle) is the 'base_link' -->
+    <!-- ================= Base Link ================= -->
     <link name="base_link">
         <inertial>
-            <mass value="${bottle_mass}" />
-            <inertia ixx="0.001" ixy="0" ixz="0" iyy="0.001" iyz="0" izz="0.001" />
+            <mass value="${bottle_mass}"/>
+            <inertia ixx="0.001" ixy="0" ixz="0" iyy="0.001" iyz="0" izz="0.001"/>
         </inertial>
         <visual>
-            <origin xyz="0 0 0" rpy="0 ${pi/2} 0" /> <!-- Rotated to lay flat -->
-            <geometry><cylinder radius="${bottle_radius}" length="${bottle_length}" /></geometry>
-            <material name="bottle_material"><color rgba="0.6 0.8 1.0 0.7" /></material> <!-- Translucent blue -->
+            <origin xyz="0 0 0" rpy="0 ${pi/2} 0"/>
+            <geometry><cylinder radius="${bottle_radius}" length="${bottle_length}"/></geometry>
+            <material name="bottle_material"><color rgba="0.6 0.8 1.0 0.7"/></material>
         </visual>
         <collision>
-            <origin xyz="0 0 0" rpy="0 ${pi/2} 0" />
-            <geometry><cylinder radius="${bottle_radius}" length="${bottle_length}" /></geometry>
+            <origin xyz="0 0 0" rpy="0 ${pi/2} 0"/>
+            <geometry><cylinder radius="${bottle_radius}" length="${bottle_length}"/></geometry>
         </collision>
     </link>
-    <!-- Rear Wheel Links -->
+    <!-- ================= Wheels ================= -->
     <xacro:macro name="wheel_link" params="prefix">
         <link name="${prefix}_wheel_link">
             <inertial>
-                <mass value="${wheel_mass}" />
-                <inertia ixx="0.0001" ixy="0" ixz="0" iyy="0.0001" iyz="0" izz="0.0001" />
+                <mass value="${wheel_mass}"/>
+                <inertia ixx="0.0001" ixy="0" ixz="0" iyy="0.0001" iyz="0" izz="0.0001"/>
             </inertial>
             <visual>
-                <origin xyz="0 0 0" rpy="${pi/2} 0 0" />
-                <geometry><cylinder radius="${wheel_radius}" length="${wheel_thickness}" /></geometry>
-                <material name="wheel_material"><color rgba="0.2 0.2 0.2 1.0" /></material>
+                <origin xyz="0 0 0" rpy="${pi/2} 0 0"/>
+                <geometry><cylinder radius="${wheel_radius}" length="${wheel_thickness}"/></geometry>
+                <material name="wheel_material"><color rgba="0.2 0.2 0.2 1.0"/></material>
             </visual>
             <collision>
-                <origin xyz="0 0 0" rpy="${pi/2} 0 0" />
-                <geometry><cylinder radius="${wheel_radius}" length="${wheel_thickness}" /></geometry>
+                <origin xyz="0 0 0" rpy="${pi/2} 0 0"/>
+                <geometry><cylinder radius="${wheel_radius}" length="${wheel_thickness}"/></geometry>
             </collision>
         </link>
@@ -48,51 +46,105 @@
     <xacro:wheel_link prefix="rear_left"/>
     <xacro:wheel_link prefix="rear_right"/>
-    <!-- Front Caster Wheel -->
+    <!-- ================= Caster ================= -->
     <link name="caster_link">
         <inertial>
-            <mass value="${caster_mass}" />
-            <inertia ixx="0.00005" ixy="0" ixz="0" iyy="0.00005" iyz="0" izz="0.00005" />
+            <mass value="${caster_mass}"/>
+            <inertia ixx="0.00005" ixy="0" ixz="0" iyy="0.00005" iyz="0" izz="0.00005"/>
         </inertial>
         <visual>
-            <geometry><sphere radius="${caster_radius}" /></geometry>
-            <material name="caster_material"><color rgba="0.1 0.1 0.1 1.0" /></material>
+            <geometry><sphere radius="${caster_radius}"/></geometry>
+            <material name="caster_material"><color rgba="0.1 0.1 0.1 1.0"/></material>
         </visual>
         <collision>
-            <geometry><sphere radius="${caster_radius}" /></geometry>
+            <geometry><sphere radius="${caster_radius}"/></geometry>
         </collision>
     </link>
-    <!-- ======================== JOINTS (Connecting the parts) ======================== -->
+    <!-- ================= LiDAR ================= -->
+    <link name="lidar_link">
+        <inertial>
+            <mass value="0.05"/>
+            <inertia ixx="0.0001" ixy="0" ixz="0" iyy="0.0001" iyz="0" izz="0.0001"/>
+        </inertial>
+        <visual>
+            <origin xyz="0 0 0" rpy="0 0 0"/>
+            <geometry><cylinder radius="0.02" length="0.05"/></geometry>
+            <material name="lidar_material"><color rgba="1 0 0 1"/></material>
+        </visual>
+        <collision>
+            <origin xyz="0 0 0" rpy="0 0 0"/>
+            <geometry><cylinder radius="0.02" length="0.05"/></geometry>
+        </collision>
+    </link>
+    <!-- ================= Joints ================= -->
     <joint name="rear_left_wheel_joint" type="continuous">
-        <parent link="base_link" />
-        <child link="rear_left_wheel_link" />
-        <origin xyz="-${bottle_length/2 - 0.05} ${bottle_radius + wheel_thickness/2} -0.01" rpy="0 0 0" />
-        <axis xyz="0 1 0" />
+        <parent link="base_link"/>
+        <child link="rear_left_wheel_link"/>
+        <origin xyz="-${bottle_length/2 - 0.05} ${bottle_radius + wheel_thickness/2} -0.01" rpy="0 0 0"/>
+        <axis xyz="0 1 0"/>
     </joint>
     <joint name="rear_right_wheel_joint" type="continuous">
-        <parent link="base_link" />
-        <child link="rear_right_wheel_link" />
-        <origin xyz="-${bottle_length/2 - 0.05} -${bottle_radius + wheel_thickness/2} -0.01" rpy="0 0 0" />
-        <axis xyz="0 1 0" />
+        <parent link="base_link"/>
+        <child link="rear_right_wheel_link"/>
+        <origin xyz="-${bottle_length/2 - 0.05} -${bottle_radius + wheel_thickness/2} -0.01" rpy="0 0 0"/>
+        <axis xyz="0 1 0"/>
     </joint>
     <joint name="caster_joint" type="fixed">
-        <parent link="base_link" />
-        <child link="caster_link" />
-        <origin xyz="${bottle_length/2} 0 -${bottle_radius}" rpy="0 0 0" />
+        <parent link="base_link"/>
+        <child link="caster_link"/>
+        <origin xyz="${bottle_length/2} 0 -${bottle_radius}" rpy="0 0 0"/>
     </joint>
-    <!-- ======================= GAZEBO ADDITIONS ======================= -->
-    <gazebo reference="rear_left_wheel_link"><mu1>1.0</mu1> <mu2>1.0</mu2> <material>Gazebo/Black</material></gazebo>
-    <gazebo reference="rear_right_wheel_link"><mu1>1.0</mu1> <mu2>1.0</mu2> <material>Gazebo/Black</material></gazebo>
-    <gazebo reference="caster_link"><mu1>0.0</mu1> <mu2>0.0</mu2> <material>Gazebo/Black</material></gazebo>
+    <joint name="lidar_joint" type="fixed">
+        <parent link="base_link"/>
+        <child link="lidar_link"/>
+        <origin xyz="0 0 ${bottle_radius + 0.05}" rpy="0 0 0"/>
+    </joint>
+    <!-- ================= Gazebo Materials ================= -->
+    <gazebo reference="rear_left_wheel_link"><mu1>1.0</mu1><mu2>1.0</mu2><material>Gazebo/Black</material></gazebo>
+    <gazebo reference="rear_right_wheel_link"><mu1>1.0</mu1><mu2>1.0</mu2><material>Gazebo/Black</material></gazebo>
+    <gazebo reference="caster_link"><mu1>0.0</mu1><mu2>0.0</mu2><material>Gazebo/Black</material></gazebo>
+    <!-- ================= Differential Drive ================= -->
     <gazebo>
         <plugin name="differential_drive_controller" filename="libgazebo_ros_diff_drive.so">
-            <alwaysOn>true</alwaysOn>
+            <rosDebugLevel>info</rosDebugLevel>
             <leftJoint>rear_left_wheel_joint</leftJoint>
             <rightJoint>rear_right_wheel_joint</rightJoint>
-            <wheelSeparation>${(bottle_radius + wheel_thickness/2) * 2}</wheelSeparation>
-            <wheelDiameter>${wheel_radius * 2}</wheelDiameter>
+            <wheelSeparation>0.1</wheelSeparation>
+            <wheelDiameter>0.06</wheelDiameter>
             <torque>20</torque>
             <commandTopic>cmd_vel</commandTopic>
+            <odometryTopic>odom</odometryTopic>
+            <odometryFrame>odom</odometryFrame>
             <robotBaseFrame>base_link</robotBaseFrame>
+            <publishWheelTF>true</publishWheelTF>
+            <publishOdomTF>true</publishOdomTF>
+            <publishWheelJointState>true</publishWheelJointState>
         </plugin>
     </gazebo>
+    <!-- ================= LiDAR Sensor Plugin ================= -->
+    <gazebo reference="lidar_link">
+        <sensor type="ray" name="lidar_sensor">
+            <pose>0 0 0 0 0 0</pose>
+            <visualize>true</visualize>
+            <update_rate>10</update_rate>
+            <ray>
+                <scan>
+                    <horizontal>
+                        <samples>360</samples>
+                        <resolution>1</resolution>
+                        <min_angle>-1.5708</min_angle>
+                        <max_angle>1.5708</max_angle>
+                    </horizontal>
+                </scan>
+                <range>
+                    <min>0.05</min>
+                    <max>10.0</max>
+                    <resolution>0.01</resolution>
+                </range>
+            </ray>
+            <plugin name="gazebo_ros_laser" filename="libgazebo_ros_laser.so">
+                <topicName>/scan</topicName>
+                <frameName>lidar_link</frameName>
+            </plugin>
+        </sensor>
+    </gazebo>
 </robot>
